File: _autosave-5.0mustangProteusPnP.sch (KiCad schematic (older format))
At the start: 7 parts, among them J1 5-146280-3, J2 5103308-3, J3 776228-1, J4 5103308-3, J5 776231-2, J6 776231-1, U1 FORD60PIN

Commit message: fixed 12V and IAC
Parts:
- removed J1: 5-146280-3, footprints:5-146280-3, symbol 2021-01-09_18-59-59:5-146280-3
- added J1: 5-146280-3, 5-146280-3:5-146280-3, symbol 5-146280-3:5-146280-3
Changed lines of the file:
@@
 Wire Notes Line
 	700  7250 700  550
-$Comp
-L 2021-01-09_18-59-59:5-146280-3 J1
-U 1 1 600203B1
-P 8650 5300
-F 0 "J1" H 9178 5253 60  0000 L CNN
-F 1 "5-146280-3" H 9178 5147 60  0000 L CNN
-F 2 "footprints:5-146280-3" H 9050 5140 60  0001 C CNN
-F 3 "" H 8650 5300 60  0000 C CNN
-	1    8650 5300
-	1    0    0    -1
-$EndComp
 Wire Wire Line
 	8650 5300 8250 5300
@@
 Main Relay Connector
 NoConn ~ 1800 4100
+$Comp
+L 5-146280-3:5-146280-3 J1
+U 1 1 5FFFBBB6
+P 8650 5300
+F 0 "J1" H 9178 5253 60  0000 L CNN
+F 1 "5-146280-3" H 9178 5147 60  0000 L CNN
+F 2 "5-146280-3:5-146280-3" H 9050 5140 60  0001 C CNN
+F 3 "" H 8650 5300 60  0000 C CNN
+	1    8650 5300
+	1    0    0    -1
+$EndComp
 $EndSCHEMATC
